File: Session1/MyBenchBuddy/KiCad/Thermocouple.sch (KiCad schematic (older format))
At the start: 0 parts

Commit message: Module2Unit11
Changed lines of the file:
@@
 Comment4 ""
 $EndDescr
-Text HLabel 6950 5650 2    60   Input ~ 0
+Text HLabel 9700 2250 2    60   Input ~ 0
 TC_IN+
-Text HLabel 7000 6200 2    60   Input ~ 0
+Text HLabel 9750 2800 2    60   Input ~ 0
 TC_IN-
+Text HLabel 1550 1750 0    60   Input ~ 0
+MOSI
+Text HLabel 1450 2000 0    60   Output ~ 0
+MISO
+Text HLabel 1450 2400 0    60   Input ~ 0
+SCLK
+Text HLabel 1400 2850 0    60   Input ~ 0
+CS_N
 $EndSCHEMATC

Commit message: Module3Unit3
Parts:
- added C?: C, symbol C
- added D?: ZENER, symbol ZENER
- added R? (x7): R, symbol R
- added U? (x4): LM324, symbol LM324
- added U? (x2): MCP3550-60-E/SN, SO8, symbol MCP3550-60-E/SN
Connections:
- net CS_N: now also U?.7 (~CS~)
- net MISO: now also U?.6 (SDO/~RDY~)
- net SCLK: now also U?.5 (SCK)
- net TC_IN+: now also U?.3 (+)
- net TC_IN-: now also U?.3 (+)
- new net: R?.1, R?.2, U?.1
- new net: R?.1, R?.2, U?.2 (-) (x3)
- new net: R?.2, R?.2, U?.1
- new net: R?.1, U?.1, U?.2 (Vin+)
- new net: R?.1, R?.2, U?.3 (+)
- new net: U?.1, U?.2 (-), U?.2 (Vin+)
- new net +12V: D?.2 (K), U?.3 (+), U?.4 (V+), U?.4 (V+), U?.4 (V+)
- new net -12V: U?.11 (V-), U?.11 (V-), U?.11 (V-)
- new net AGND: D?.1 (A), R?.1, U?.3 (Vin-), U?.3 (Vin-)
Other:
- note added: "16-24bit ADC"
- note added: "Analog/TC Input"
- note added: "General temperature sensor."
- note added: "Instrumentation Amp"
