File: Session1A/MyBenchBuddy/MyBenchBuddy.sch (KiCad schematic (older format))
At the start: 0 parts

Commit message: Defining Your Inputs and Outputs
Changed lines of the file:
@@
 Sheet 1 8
 Title ""
-Date "3 feb 2014"
+Date "4 feb 2014"
 Rev ""
 Comp ""
@@
 $EndDescr
 $Sheet
-S 1000 4950 2200 2100
+S 1200 3650 2450 3550
 U 52EF36BC
 F0 "Arduino" 50
 F1 "Arduino.sch" 50
+F2 "Relay+" O R 3650 6600 60
+F3 "Relay-" I R 3650 6750 60
+F4 "MOSI" O R 3650 5600 60
+F5 "MISO" I R 3650 5750 60
+F6 "SCLK" O R 3650 5900 60
+F7 "CS_N" O R 3650 6050 60
+F8 "LED_EN" O R 3650 5000 60
+F9 "LED_FREQ" O R 3650 5150 60
+F10 "FAN_EN" O R 3650 4500 60
+F11 "TACH_MEAS" I R 3650 4650 60
 $EndSheet
 $Sheet
@@
 F2 "TC IN +" I R 9300 4450 60
 F3 "TC IN -" I R 9300 4650 60
+F4 "MOSI" I L 7550 4400 60
+F5 "MISO" O L 7550 4550 60
+F6 "SCLK" I L 7550 4700 60
+F7 "CS_N" I L 7550 4850 60
 $EndSheet
 $Sheet
@@
 F0 "Relay" 50
 F1 "Relay.sch" 50
+F2 "DIN+" I L 7550 5850 60
+F3 "DIN-" O L 7550 6050 60
+F4 "Relay+" I R 9250 5850 60
+F5 "Relay-" O R 9250 6000 60
 $EndSheet
 $Sheet
@@
 F0 "LED_Driver" 50
 F1 "LED_Driver.sch" 50
+F2 "EN" I L 7550 2800 60
+F3 "FREQ" I L 7550 3000 60
+F4 "String+" O R 9300 2750 60
+F5 "String-" I R 9300 2950 60
 $EndSheet
 $Sheet
@@
 F0 "Fan" 50
 F1 "Fan.sch" 50
+F2 "Power+" O R 9450 1050 60
+F3 "Power-" I R 9450 1200 60
+F4 "Tach" I R 9450 1350 60
+F5 "Tach_out" O L 7550 1300 60
+F6 "Fan_In" I L 7550 1050 60
 $EndSheet
 $Sheet

Commit message: Understanding The Current/Fan Driver Module
Changed lines of the file:
@@
 Sheet 1 8
 Title ""
-Date "5 feb 2014"
+Date "9 feb 2014"
 Rev ""
 Comp ""
@@
 F3 "Power-" I R 9450 1200 60
 F4 "Tach" I R 9450 1350 60
-F5 "Tach_out" O L 7550 1300 60
+F5 "Tach_out" O L 7550 2100 60
 F6 "Fan_In" I L 7550 1050 60
+F7 "Current Measure" O L 7550 1950 60
+F8 "MOSI" I L 7550 1300 60
+F9 "MISO" O L 7550 1400 60
+F10 "CS_N" I L 7550 1500 60
+F11 "SCLK" I L 7550 1600 60
 $EndSheet
 $Sheet

Commit message: Understanding The Power Protection and Filtering Module
Changed lines of the file:
@@
 LIBS:valves
 LIBS:bth-switch
+LIBS:bth-power
 LIBS:MyBenchBuddy-cache
 EELAYER 27 0
@@
 $Descr A4 11693 8268
 encoding utf-8
-Sheet 1 8
+Sheet 1 9
 Title ""
-Date "9 feb 2014"
+Date "11 feb 2014"
 Rev ""
 Comp ""
@@
 F1 "TerminalBlock.sch" 50
 $EndSheet
+$Sheet
+S 3850 900  2350 1300
+U 52F9B182
+F0 "PowerAdjustmentMonitor" 50
+F1 "PowerAdjustmentMonitor.sch" 50
+$EndSheet
 $EndSCHEMATC
