File: Session1A/MyBenchBuddy/Thermocouple.sch (KiCad schematic (older format))
At the start: 15 parts

Commit message: initial
Parts:
- removed D?: ZENER, ~, symbol ZENER
- removed U?: LM324, symbol LM324
- removed U? (x2): MCP3550-60-E/SN, SO8, symbol MCP3550-60-E/SN
- added C10, C6, C7, C8, C9: C, ~, symbol C
- added P2: CONN_3X2, symbol CONN_3X2
- added P3: CONN_2, symbol CONN_2
- added R42, R43: R, ~, symbol R
- added U10: LMT84, symbol LMT84
- added U9: MCP3901, symbol MCP3901
- U11: renamed from U?; value LM324 -> OPA4170
- gave numbers to parts that had none: 8
Connections:
- net +12V: now also C10.2
- net -12V: now also C9.2
- net AGND: now also C5.2, C10.1, C6.2, C7.2, C8.2, C9.1, U10.1 (GND), U10.2 (GND), U10.5 (GND), U9.11 (DGND), U9.5 (CH0-), U9.6 (CH1-), U9.8 (AGND)
- net MISO: now also U9.19 (SDO)
- net MOSI: now also U9.20 (SDI)
- net SCLK: now also U9.18 (SCK)
- net TC IN +: now also U11.5 (+); no longer U11.3 (+)
- net TC IN -: now also U11.10 (+); no longer U11.3 (+)
- net at R37.2, R39.1: now also U11.7; no longer U11.1
- net at R38.2, R41.2: now also U11.8; no longer U11.1
- net at R40.2, R41.1: now also U11.9 (-), R42.2, R43.2; no longer U11.2 (-)
- net at R35.1: now also C5.1, U11.14, U9.4 (CH0+); no longer U11.1
- net at R35.2, R37.1: now also U11.13 (-); no longer U11.2 (-)
- net at R36.2, R38.1: now also U11.12 (+); no longer U11.3 (+)
- new net: P2.1, P2.3, P2.5, R39.2, U11.6 (-)
- new net: P2.6, R40.1
- new net: P3.1 (P1), U9.12 (MDAT1)
- new net: P3.2 (PM), U9.13 (MDAT0)
- new net: U10.3 (OUT), U9.7 (CH1+)
- new net: P2.4, R42.1
- new net: P2.2, R43.1
- new net +5V: C6.1, C7.1, C8.1, U10.4 (Vdd), U9.2 (DVdd), U9.3 (AVdd)
- new net REF+: U9.9 (REFINOUT+)
- new net REF-: U9.10 (REFIN-)
- new net ~CS: U9.17 (~CS)
- new net ~DR: U9.14 (~DR)
- new net ~RESET: U9.1 (~RESET)
Other:
- note added: "TEMP SENSOR"
- note removed: "General\nTemperature\nSensor"
- moved on the sheet: C5, R39, R40, R41
