File: Session1A/MyBenchBuddy/MyBenchBuddy.kicad_pcb (KiCad board)
At the start: 2 copper layers, 0 parts

Commit message: initial
Parts:
- added D1: LG Q971-KN-1, LED-0603, F.Cu at (265.1, 104.3)
- added D2: B130-13-F, SMA, F.Cu at (264.4, 112.5)
- added K1: 1461069-5, TE-ORWH-RELAY, F.Cu at (270.3, 104.2)
- added Q1: 2N3904, SOT23EBC, B.Cu at (268.8, 110.8)
- added R1: 500, SM0805, B.Cu at (253.0, 99.5)
- added R2: 200, SM0805, B.Cu at (261.8, 104.5)
- added R3: 100, SM0805, F.Cu at (257.9, 103.9)
- added R4: 0, SM0805, B.Cu at (269.3, 101.0)
- added R5: 0, SM0805, F.Cu at (268.8, 97.1)
- added R6: 0, SM0805, B.Cu at (273.5, 113.3)
- added U1: LTV-816S, 4-SMD, F.Cu at (256.0, 98.1)
Other:
- board outline added: 165.1 x 63.5 mm
