File: Session1A/MyBenchBuddy/PowerAdjustmentMonitor.sch (KiCad schematic (older format))
At the start: 19 parts

Commit message: initial
Parts:
- gave numbers to parts that had none: 18
Changed lines of the file:
@@
 Sheet 5 9
 Title ""
-Date "1 mar 2014"
+Date "15 mar 2014"
 Rev ""
 Comp ""
@@
 $EndDescr
 $Comp
-L +3.3V #PWR?
+L +3.3V #PWR30
 U 1 1 52FACA77
 P 6100 3250
-F 0 "#PWR?" H 6100 3210 30  0001 C CNN
+F 0 "#PWR30" H 6100 3210 30  0001 C CNN
 F 1 "+3.3V" H 6100 3360 30  0000 C CNN
 F 2 "" H 6100 3250 60  0000 C CNN
@@
 $EndComp
 $Comp
-L +5V #PWR?
+L +5V #PWR29
 U 1 1 52FACA7D
 P 5850 3250
-F 0 "#PWR?" H 5850 3340 20  0001 C CNN
+F 0 "#PWR29" H 5850 3340 20  0001 C CNN
 F 1 "+5V" H 5850 3340 30  0000 C CNN
 F 2 "" H 5850 3250 60  0000 C CNN
@@
 $EndComp
 $Comp
-L +12V #PWR?
+L +12V #PWR22
 U 1 1 52FACB0A
 P 1600 3250
-F 0 "#PWR?" H 1600 3200 20  0001 C CNN
+F 0 "#PWR22" H 1600 3200 20  0001 C CNN
 F 1 "+12V" H 1600 3350 30  0000 C CNN
 F 2 "" H 1600 3250 60  0000 C CNN
@@
 $EndComp
 $Comp
-L -12V #PWR?
+L -12V #PWR23
 U 1 1 52FACB12
 P 1600 5100
-F 0 "#PWR?" H 1600 5230 20  0001 C CNN
+F 0 "#PWR23" H 1600 5230 20  0001 C CNN
 F 1 "-12V" H 1600 5200 30  0000 C CNN
 F 2 "" H 1600 5100 60  0000 C CNN
@@
 $EndComp
 $Comp
-L LM317 U?
+L LM317 U4
 U 1 1 52FAD064
 P 2400 7200
-F 0 "U?" H 2400 7500 60  0000 C CNN
+F 0 "U4" H 2400 7500 60  0000 C CNN
 F 1 "LM317" H 2450 6950 60  0000 L CNN
 F 2 "~" H 2400 7200 60  0000 C CNN
@@
 $EndComp
 $Comp
-L JUMPER JP?
+L JUMPER JP3
 U 1 1 52FAD417
 P 2450 5350
-F 0 "JP?" H 2450 5500 60  0000 C CNN
+F 0 "JP3" H 2450 5500 60  0000 C CNN
 F 1 "JUMPER" H 2450 5270 40  0000 C CNN
 F 2 "~" H 2450 5350 60  0000 C CNN
@@
 $EndComp
 $Comp
-L JUMPER JP?
+L JUMPER JP2
 U 1 1 52FAD426
 P 2450 3050
-F 0 "JP?" H 2450 3200 60  0000 C CNN
+F 0 "JP2" H 2450 3200 60  0000 C CNN
 F 1 "JUMPER" H 2450 2970 40  0000 C CNN
 F 2 "~" H 2450 3050 60  0000 C CNN
@@
 $EndComp
 $Comp
-L GND #PWR?
+L GND #PWR20
 U 1 1 52FAD64E
 P 900 4500
-F 0 "#PWR?" H 900 4500 30  0001 C CNN
+F 0 "#PWR20" H 900 4500 30  0001 C CNN
 F 1 "GND" H 900 4430 30  0001 C CNN
 F 2 "" H 900 4500 60  0000 C CNN
@@
 $EndComp
 $Comp
-L AGND #PWR?
+L AGND #PWR21
 U 1 1 52FAD841
 P 1500 4500
-F 0 "#PWR?" H 1500 4500 40  0001 C CNN
+F 0 "#PWR21" H 1500 4500 40  0001 C CNN
 F 1 "AGND" H 1500 4430 50  0000 C CNN
 F 2 "" H 1500 4500 60  0000 C CNN
@@
 $EndComp
 $Comp
-L JUMPER JP?
+L JUMPER JP1
 U 1 1 52FAD84E
 P 1200 4150
-F 0 "JP?" H 1200 4300 60  0000 C CNN
+F 0 "JP1" H 1200 4300 60  0000 C CNN
 F 1 "JUMPER" H 1200 4070 40  0000 C CNN
 F 2 "~" H 1200 4150 60  0000 C CNN
@@
 $EndComp
 $Comp
-L AGND #PWR?
+L AGND #PWR24
 U 1 1 52FAD872
 P 2000 4400
-F 0 "#PWR?" H 2000 4400 40  0001 C CNN
+F 0 "#PWR24" H 2000 4400 40  0001 C CNN
 F 1 "AGND" H 2000 4330 50  0000 C CNN
 F 2 "" H 2000 4400 60  0000 C CNN
@@
 $EndComp
 $Comp
-L FE_V+ #PWR?
+L FE_V+ #PWR27
 U 1 1 52FADC57
 P 3050 2900
-F 0 "#PWR?" H 3050 3000 30  0001 C CNN
+F 0 "#PWR27" H 3050 3000 30  0001 C CNN
 F 1 "FE_V+" H 3050 3000 30  0000 C CNN
 F 2 "" H 3050 2900 60  0000 C CNN
@@
 $EndComp
 $Comp
-L FE_V- #PWR?
+L FE_V- #PWR28
 U 1 1 52FADE62
 P 3100 5600
-F 0 "#PWR?" H 3100 5800 40  0001 C CNN
+F 0 "#PWR28" H 3100 5800 40  0001 C CNN
 F 1 "FE_V-" H 3100 5750 40  0000 C CNN
 F 2 "" H 3100 5600 60  0000 C CNN
@@
 $EndComp
 $Comp
-L 7805 U?
+L 7805 U5
 U 1 1 52FAE280
 P 2450 3500
-F 0 "U?" H 2600 3304 60  0000 C CNN
+F 0 "U5" H 2600 3304 60  0000 C CNN
 F 1 "7805" H 2450 3700 60  0000 C CNN
 F 2 "~" H 2450 3500 60  0000 C CNN
@@
 $EndComp
 $Comp
-L 7805 U?
+L 7805 U6
 U 1 1 52FAE28F
 P 2450 4850
-F 0 "U?" H 2600 4654 60  0000 C CNN
+F 0 "U6" H 2600 4654 60  0000 C CNN
 F 1 "7805" H 2450 5050 60  0000 C CNN
 F 2 "~" H 2450 4850 60  0000 C CNN
@@
 $EndComp
 $Comp
-L R R?
+L R R11
 U 1 1 52FAE940
 P 2950 6450
-F 0 "R?" V 3030 6450 40  0000 C CNN
+F 0 "R11" V 3030 6450 40  0000 C CNN
 F 1 "R" V 2957 6451 40  0000 C CNN
 F 2 "~" V 2880 6450 30  0000 C CNN
@@
 $EndComp
 $Comp
-L AGND #PWR?
+L AGND #PWR25
 U 1 1 52FAEC11
 P 2650 6150
-F 0 "#PWR?" H 2650 6150 40  0001 C CNN
+F 0 "#PWR25" H 2650 6150 40  0001 C CNN
 F 1 "AGND" H 2650 6080 50  0000 C CNN
 F 2 "" H 2650 6150 60  0000 C CNN
@@
 $EndComp
 $Comp
-L LM317 U?
+L LM317 U3
 U 1 1 52FAF069
 P 2300 1250
-F 0 "U?" H 2300 1550 60  0000 C CNN
+F 0 "U3" H 2300 1550 60  0000 C CNN
 F 1 "LM317" H 2350 1000 60  0000 L CNN
 F 2 "~" H 2300 1250 60  0000 C CNN
@@
 $EndComp
 $Comp
-L R R?
+L R R10
 U 1 1 52FAF076
 P 2850 2000
-F 0 "R?" V 2930 2000 40  0000 C CNN
+F 0 "R10" V 2930 2000 40  0000 C CNN
 F 1 "R" V 2857 2001 40  0000 C CNN
 F 2 "~" V 2780 2000 30  0000 C CNN
@@
 $EndComp
 $Comp
-L AGND #PWR?
+L AGND #PWR26
 U 1 1 52FAF082
 P 2850 2400
-F 0 "#PWR?" H 2850 2400 40  0001 C CNN
+F 0 "#PWR26" H 2850 2400 40  0001 C CNN
 F 1 "AGND" H 2850 2330 50  0000 C CNN
 F 2 "" H 2850 2400 60  0000 C CNN
@@
 V-_CURR_MON
 $Comp
-L R R?
+L R R16
 U 1 1 52FB05B3
 P 4800 3600
-F 0 "R?" V 4880 3600 40  0000 C CNN
+F 0 "R16" V 4880 3600 40  0000 C CNN
 F 1 "R" V 4807 3601 40  0000 C CNN
 F 2 "~" V 4730 3600 30  0000 C CNN
@@
 $EndComp
 $Comp
-L R R?
+L R R15
 U 1 1 52FB05C0
 P 4800 2900
-F 0 "R?" V 4880 2900 40  0000 C CNN
+F 0 "R15" V 4880 2900 40  0000 C CNN
 F 1 "R" V 4807 2901 40  0000 C CNN
 F 2 "~" V 4730 2900 30  0000 C CNN
@@
 $EndComp
 $Comp
-L R R?
+L R R17
 U 1 1 52FB0653
 P 4800 4700
-F 0 "R?" V 4880 4700 40  0000 C CNN
+F 0 "R17" V 4880 4700 40  0000 C CNN
 F 1 "R" V 4807 4701 40  0000 C CNN
 F 2 "~" V 4730 4700 30  0000 C CNN
@@
 $EndComp
 $Comp
-L R R?
+L R R18
 U 1 1 52FB0659
 P 4800 5400
-F 0 "R?" V 4880 5400 40  0000 C CNN
+F 0 "R18" V 4880 5400 40  0000 C CNN
 F 1 "R" V 4807 5401 40  0000 C CNN
 F 2 "~" V 4730 5400 30  0000 C CNN
@@
 	5850 3600 5850 3250
 $Comp
-L R R?
+L R R14
 U 1 1 52FB1374
 P 3400 7350
-F 0 "R?" V 3480 7350 40  0000 C CNN
+F 0 "R14" V 3480 7350 40  0000 C CNN
 F 1 "R" V 3407 7351 40  0000 C CNN
 F 2 "~" V 3330 7350 30  0000 C CNN
@@
 	3650 7350 4250 7350
 $Comp
-L R R?
+L R R13
 U 1 1 52FB1699
 P 3300 1100
-F 0 "R?" V 3380 1100 40  0000 C CNN
+F 0 "R13" V 3380 1100 40  0000 C CNN
 F 1 "R" V 3307 1101 40  0000 C CNN
 F 2 "~" V 3230 1100 30  0000 C CNN
@@
 V+_MON
 $Comp
-L LM324 U?
+L LM324 U7
 U 1 1 52FB1CA3
 P 8850 4800
-F 0 "U?" H 8900 5000 60  0000 C CNN
+F 0 "U7" H 8900 5000 60  0000 C CNN
 F 1 "LM324" H 9000 4600 50  0000 C CNN
 F 2 "" H 8850 4800 60  0000 C CNN
@@
 $EndComp
 $Comp
-L +12V #PWR?
+L +12V #PWR31
 U 1 1 52FB1CBE
 P 8750 4250
-F 0 "#PWR?" H 8750 4200 20  0001 C CNN
+F 0 "#PWR31" H 8750 4200 20  0001 C CNN
 F 1 "+12V" H 8750 4350 30  0000 C CNN
 F 2 "" H 8750 4250 60  0000 C CNN
@@
 $EndComp
 $Comp
-L -12V #PWR?
+L -12V #PWR32
 U 1 1 52FB1EE3
 P 8750 5300
-F 0 "#PWR?" H 8750 5430 20  0001 C CNN
+F 0 "#PWR32" H 8750 5430 20  0001 C CNN
 F 1 "-12V" H 8750 5400 30  0000 C CNN
 F 2 "" H 8750 5300 60  0000 C CNN
@@
 	8750 4250 8750 4400
 $Comp
-L LM324 U?
-U 1 1 52FB21EE
+L LM324 U7
+U 2 1 52FB21EE
 P 8850 6400
-F 0 "U?" H 8900 6600 60  0000 C CNN
+F 0 "U7" H 8900 6600 60  0000 C CNN
 F 1 "LM324" H 9000 6200 50  0000 C CNN
 F 2 "" H 8850 6400 60  0000 C CNN
 F 3 "" H 8850 6400 60  0000 C CNN
-	1    8850 6400
-	1    0    0    -1
-$EndComp
-$Comp
-L +12V #PWR?
+	2    8850 6400
+	1    0    0    -1
+$EndComp
+$Comp
+L +12V #PWR33
 U 1 1 52FB21F4
 P 8750 5850
-F 0 "#PWR?" H 8750 5800 20  0001 C CNN
+F 0 "#PWR33" H 8750 5800 20  0001 C CNN
 F 1 "+12V" H 8750 5950 30  0000 C CNN
 F 2 "" H 8750 5850 60  0000 C CNN
@@
 $EndComp
 $Comp
-L -12V #PWR?
+L -12V #PWR34
 U 1 1 52FB21FA
 P 8750 6900
-F 0 "#PWR?" H 8750 7030 20  0001 C CNN
+F 0 "#PWR34" H 8750 7030 20  0001 C CNN
 F 1 "-12V" H 8750 7000 30  0000 C CNN
 F 2 "" H 8750 6900 60  0000 C CNN
@@
 V+_MON
 $Comp
-L RVAR R?
+L RVAR R12
 U 1 1 52FB33D2
 P 2950 7100
-F 0 "R?" V 3030 7050 50  0000 C CNN
+F 0 "R12" V 3030 7050 50  0000 C CNN
 F 1 "RVAR" V 2870 7160 50  0000 C CNN
 F 2 "~" H 2950 7100 60  0000 C CNN
@@
 $EndComp
 $Comp
-L RVAR R?
+L RVAR R9
 U 1 1 52FB35F1
 P 2850 1350
-F 0 "R?" V 2930 1300 50  0000 C CNN
+F 0 "R9" V 2930 1300 50  0000 C CNN
 F 1 "RVAR" V 2770 1410 50  0000 C CNN
 F 2 "~" H 2850 1350 60  0000 C CNN
