File: FullChargeAhead/pcb/FullChargeAhead.sch (KiCad schematic (older format))
At the start: 18 parts, among them CON101 USB-MICRO-B, P101 TIMER, P102 BATT, U101 MCP73834-FCI/UN

Commit message: FCA final footprints and initial pcb layout w/out wires
Parts:
- C101, C102: footprint (none) -> Capacitors_SMD:C_0805_HandSoldering
- D102, D103: footprint (none) -> LEDs:LED-0805
- P101: footprint (none) -> Pin_Headers:Pin_Header_Straight_1x02
- P102: footprint (none) -> pcb:JST_2pin_lipo_S2B-PH-SM4-TB
- TH101: footprint (none) -> Resistors_SMD:R_0805_HandSoldering
- U101: footprint (none) -> pcb:MSOP-10
Changed lines of the file:
@@
 F 0 "U101" H 6650 2850 60  0000 C CNN
 F 1 "MCP73834-FCI/UN" V 6400 3400 60  0000 C CNN
-F 2 "" H 6500 3350 60  0001 C CNN
+F 2 "pcb:MSOP-10" H 6500 3350 60  0001 C CNN
 F 3 "" H 6500 3350 60  0000 C CNN
 	1    6350 3400
@@
 F 0 "C101" H 3900 3150 50  0000 L CNN
 F 1 "4.7uf" H 3900 2950 50  0000 L CNN
-F 2 "" H 3888 2900 30  0001 C CNN
+F 2 "Capacitors_SMD:C_0805_HandSoldering" H 3888 2900 30  0001 C CNN
 F 3 "" H 3850 3050 60  0000 C CNN
 F 4 "Value" H 3850 3050 60  0001 C CNN "MPN"
@@
 F 0 "C102" H 7950 3400 50  0000 L CNN
 F 1 "4.7uf" H 7950 3200 50  0000 L CNN
-F 2 "" H 7938 3150 30  0001 C CNN
+F 2 "Capacitors_SMD:C_0805_HandSoldering" H 7938 3150 30  0001 C CNN
 F 3 "" H 7900 3300 60  0000 C CNN
 F 4 "Value" H 7900 3300 60  0001 C CNN "MPN"
@@
 F 0 "TH101" V 7800 3950 50  0000 C CNN
 F 1 "10K" V 7600 3900 50  0000 C BNN
-F 2 "" H 7700 3900 60  0001 C CNN
+F 2 "Resistors_SMD:R_0805_HandSoldering" H 7700 3900 60  0001 C CNN
 F 3 "" H 7700 3900 60  0000 C CNN
 F 4 "Value" H 7700 3900 60  0001 C CNN "MPN"
@@
 F 0 "D103" H 5050 3150 50  0000 C CNN
 F 1 "LED" H 5050 2950 50  0000 C CNN
-F 2 "" H 5050 3050 60  0001 C CNN
+F 2 "LEDs:LED-0805" H 5050 3050 60  0001 C CNN
 F 3 "" H 5050 3050 60  0000 C CNN
 	1    5050 3050
@@
 F 0 "D102" H 4650 3150 50  0000 C CNN
 F 1 "LED" H 4650 2950 50  0000 C CNN
-F 2 "" H 4650 3050 60  0001 C CNN
+F 2 "LEDs:LED-0805" H 4650 3050 60  0001 C CNN
 F 3 "" H 4650 3050 60  0000 C CNN
 	1    4650 3050
@@
 F 0 "P102" H 8750 3550 50  0000 C CNN
 F 1 "BATT" V 8850 3400 50  0000 C CNN
-F 2 "" H 8750 3400 60  0001 C CNN
+F 2 "pcb:JST_2pin_lipo_S2B-PH-SM4-TB" H 8750 3400 60  0001 C CNN
 F 3 "" H 8750 3400 60  0000 C CNN
 	1    8750 3400
@@
 F 0 "P101" H 5700 4700 50  0000 C CNN
 F 1 "TIMER" V 5800 4550 50  0000 C CNN
-F 2 "" H 5700 4550 60  0001 C CNN
+F 2 "Pin_Headers:Pin_Header_Straight_1x02" H 5700 4550 60  0001 C CNN
 F 3 "" H 5700 4550 60  0000 C CNN
 	1    5700 4550

Commit message: First board layout complete and initial gerbers.
Parts:
- removed TH101: 10K, Resistors_SMD:R_0805_HandSoldering, symbol THERMISTOR
- added P103, P104, P105, P106: CONN_01X01, Connect:1pin, symbol CONN_01X01
- added P107: THERM, Pin_Headers:Pin_Header_Straight_1x02, symbol CONN_01X02
- added R109: 1.54K, Resistors_SMD:R_0805_HandSoldering, symbol R
- added R110: 69.8K, Resistors_SMD:R_0805_HandSoldering, symbol R
- CON101: footprint (none) -> pcb:MICRO_B_CONN_10118193-0001LF
- D101: footprint (none) -> LEDs:LED-0805
Connections:
- net GND: now also P107.2 (P2), R110.2
- net Vdd: now reaches C101.1, CON101.1 (VBUS), D101.1 (A), D102.1 (A), D103.1 (A), U101.1 (VDD), U101.2 (VDD)
- net Vbat: now reaches C102.1, P102.1 (P1), U101.10 (VBAT), U101.9 (VBAT)
- net at U101.8 (THERM): now also R109.1
- new net: P107.1 (P1), R109.2, R110.1
- no-connect marks 0 -> 4
Changed lines of the file:
@@
 LIBS:contrib
 LIBS:valves
-LIBS:FullChargeAhead
-LIBS:FullChargeAhead-cache
+LIBS:alphaomega
+LIBS:trenchmos
+LIBS:sink_or_swim-cache
 EELAYER 25 0
 EELAYER END
@@
 $EndComp
 $Comp
-L THERMISTOR TH101
-U 1 1 5508CCB7
-P 7700 3900
-F 0 "TH101" V 7800 3950 50  0000 C CNN
-F 1 "10K" V 7600 3900 50  0000 C BNN
-F 2 "Resistors_SMD:R_0805_HandSoldering" H 7700 3900 60  0001 C CNN
-F 3 "" H 7700 3900 60  0000 C CNN
-F 4 "Value" H 7700 3900 60  0001 C CNN "MPN"
-	1    7700 3900
-	1    0    0    -1
-$EndComp
-$Comp
 L R R105
 U 1 1 5508CD13
@@
 Wire Wire Line
 	7050 3400 7700 3400
-Wire Wire Line
-	7700 3400 7700 3650
-Wire Wire Line
-	7700 4150 7700 4300
 $Comp
 L GND #PWR03
 U 1 1 5508D878
-P 7700 4300
-F 0 "#PWR03" H 7700 4050 60  0001 C CNN
-F 1 "GND" H 7700 4150 60  0000 C CNN
-F 2 "" H 7700 4300 60  0000 C CNN
-F 3 "" H 7700 4300 60  0000 C CNN
-	1    7700 4300
+P 7700 5100
+F 0 "#PWR03" H 7700 4850 60  0001 C CNN
+F 1 "GND" H 7700 4950 60  0000 C CNN
+F 2 "" H 7700 5100 60  0000 C CNN
+F 3 "" H 7700 5100 60  0000 C CNN
+	1    7700 5100
 	1    0    0    -1
 $EndComp
@@
 F 0 "CON101" H 2250 3250 50  0000 C CNN
 F 1 "USB-MICRO-B" H 2400 2550 50  0000 C CNN
-F 2 "" H 2550 2800 50  0001 C CNN
+F 2 "pcb:MICRO_B_CONN_10118193-0001LF" H 2550 2800 50  0001 C CNN
 F 3 "" H 2550 2800 50  0000 C CNN
 	1    2550 2900
@@
 F 0 "D101" H 4300 3150 50  0000 C CNN
 F 1 "NOPOP" H 4300 2950 50  0000 C CNN
-F 2 "" H 4300 3050 60  0001 C CNN
+F 2 "LEDs:LED-0805" H 4300 3050 60  0001 C CNN
 F 3 "" H 4300 3050 60  0000 C CNN
 F 4 "Value" H 4300 3050 60  0001 C CNN "MPN"
@@
 	3600 3000 3700 3000
 Connection ~ 3700 3000
+$Comp
+L CONN_01X01 P103
+U 1 1 550C6639
+P 9250 2000
+F 0 "P103" H 9250 2100 50  0000 C CNN
+F 1 "CONN_01X01" V 9350 2000 50  0000 C CNN
+F 2 "Connect:1pin" H 9250 2000 60  0001 C CNN
+F 3 "" H 9250 2000 60  0000 C CNN
+	1    9250 2000
+	1    0    0    -1
+$EndComp
+NoConn ~ 9050 2000
+$Comp
+L CONN_01X01 P105
+U 1 1 550C6850
+P 9650 2000
+F 0 "P105" H 9650 2100 50  0000 C CNN
+F 1 "CONN_01X01" V 9750 2000 50  0000 C CNN
+F 2 "Connect:1pin" H 9650 2000 60  0001 C CNN
+F 3 "" H 9650 2000 60  0000 C CNN
+	1    9650 2000
+	1    0    0    -1
+$EndComp
+$Comp
+L CONN_01X01 P106
+U 1 1 550C6890
+P 9650 2550
+F 0 "P106" H 9650 2650 50  0000 C CNN
+F 1 "CONN_01X01" V 9750 2550 50  0000 C CNN
+F 2 "Connect:1pin" H 9650 2550 60  0001 C CNN
+F 3 "" H 9650 2550 60  0000 C CNN
+	1    9650 2550
+	1    0    0    -1
+$EndComp
+$Comp
+L CONN_01X01 P104
+U 1 1 550C68C7
+P 9250 2550
+F 0 "P104" H 9250 2650 50  0000 C CNN
+F 1 "CONN_01X01" V 9350 2550 50  0000 C CNN
+F 2 "Connect:1pin" H 9250 2550 60  0001 C CNN
+F 3 "" H 9250 2550 60  0000 C CNN
+	1    9250 2550
+	1    0    0    -1
+$EndComp
+NoConn ~ 9450 2000
+NoConn ~ 9450 2550
+NoConn ~ 9050 2550
+$Comp
+L R R109
+U 1 1 550EEC9B
+P 7700 3900
+F 0 "R109" V 7780 3900 50  0000 C CNN
+F 1 "1.54K" V 7707 3901 50  0000 C CNN
+F 2 "Resistors_SMD:R_0805_HandSoldering" V 7630 3900 30  0001 C CNN
+F 3 "" H 7700 3900 30  0000 C CNN
+F 4 "Value" H 7700 3900 60  0001 C CNN "MPN"
+	1    7700 3900
+	1    0    0    -1
+$EndComp
+Wire Wire Line
+	7700 3400 7700 3650
+$Comp
+L R R110
+U 1 1 550EEE49
+P 7700 4650
+F 0 "R110" V 7780 4650 50  0000 C CNN
+F 1 "69.8K" V 7707 4651 50  0000 C CNN
+F 2 "Resistors_SMD:R_0805_HandSoldering" V 7630 4650 30  0001 C CNN
+F 3 "" H 7700 4650 30  0000 C CNN
+F 4 "Value" H 7700 4650 60  0001 C CNN "MPN"
+	1    7700 4650
+	1    0    0    -1
+$EndComp
+Wire Wire Line
+	7700 4400 7700 4150
+Wire Wire Line
+	7700 4300 8550 4300
+Wire Wire Line
+	8550 4300 8550 4600
+Connection ~ 7700 4300
+$Comp
+L GND #PWR08
+U 1 1 550EF18A
+P 8550 5100
+F 0 "#PWR08" H 8550 4850 60  0001 C CNN
+F 1 "GND" H 8550 4950 60  0000 C CNN
+F 2 "" H 8550 5100 60  0000 C CNN
+F 3 "" H 8550 5100 60  0000 C CNN
+	1    8550 5100
+	1    0    0    -1
+$EndComp
+Wire Wire Line
+	7700 5100 7700 4900
+Wire Wire Line
+	8550 4700 8550 5100
+Text Label 4000 2700 0    60   ~ 0
+Vdd
+Text Label 7600 3000 0    60   ~ 0
+Vbat
+$Comp
+L CONN_01X02 P107
+U 1 1 5510ADD8
+P 8750 4650
+F 0 "P107" H 8750 4800 50  0000 C CNN
+F 1 "THERM" V 8850 4650 50  0000 C CNN
+F 2 "Pin_Headers:Pin_Header_Straight_1x02" H 8750 4650 60  0001 C CNN
+F 3 "" H 8750 4650 60  0000 C CNN
+	1    8750 4650
+	1    0    0    -1
+$EndComp
 $EndSCHEMATC
