File: DasBlinkInput/pcb/DasBlinkInput.kicad_pcb (KiCad board)
At the start: 4 copper layers, 60 x 25 mm, 34 parts, among them P101 CONN_01X02, P102 TP_VGND, P103 TP_GND, P104 TP_3V, P105 CONN_01X05, P201 TP_CHAN1, P301 TP_CHAN2, P401 TP_CHAN3, P501 TP_CHAN4, U101 LP2980-N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

Commit message: DBI : complete pcb
Parts:
- added P106: VREF, pcb:TESTPOINT_1, F.Cu at (143.5, 91.9)
- moved R501 80.9 mm to (107.9, 87.9)
- moved P501 77.6 mm to (105.0, 90.0)
- moved C501 77.5 mm to (107.7, 85.7)
- moved R202 74.4 mm to (138.8, 90.9)
- moved C401 67.5 mm to (114.3, 85.6), turned to 180 degrees
- moved R401 62.3 mm to (114.4, 87.8), turned to 180 degrees
- moved P401 58.5 mm to (118.2, 89.2)
- moved P201 58.2 mm to (128.2, 98.1)
- moved R201 56.5 mm to (107.3, 97.9)
- moved C201 56.4 mm to (119.0, 98.3), turned to 180 degrees
- moved C202 55.7 mm to (103.7, 97.3), turned to 270 degrees
- moved C203 53.6 mm to (124.3, 98.5)
- moved RV201 52.1 mm to (138.2, 96.2), turned to 90 degrees
- moved R301 41.3 mm to (118.0, 94.7), turned to 90 degrees
- moved R203 40.9 mm to (113.9, 98.5)
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Routing:
- net VGND: track 12.2 -> 68.5 mm, vias 1 -> 6
- net /Channel2Photodetect/REF_IN: track 0.00 -> 41.9 mm
- net Net-(C202-Pad1): track 0.00 -> 39.2 mm
- net Net-(C501-Pad1): track 0.00 -> 38.9 mm, vias 0 -> 2
- net Net-(C501-Pad2): track 0.00 -> 38.3 mm, vias 0 -> 1
- net /Channel4Photodetect/CHAN4_OUT: track 0.00 -> 28.4 mm
- net /Channel3Photodetect/CHAN3_OUT: track 0.00 -> 28.0 mm
- net /Channel2Photodetect/CHAN2_OUT: track 0.00 -> 27.6 mm, vias 0 -> 1
- net /Channel1Photodetect/CHAN1_OUT: track 0.00 -> 26.7 mm, vias 0 -> 1
- net Net-(C301-Pad1): track 0.00 -> 24.5 mm, vias 0 -> 2
- net Net-(C202-Pad2): track 0.00 -> 23.4 mm, vias 0 -> 1
- net Net-(C401-Pad1): track 0.00 -> 22.7 mm, vias 0 -> 2
- net Net-(R203-Pad2): track 0.00 -> 21.8 mm
- net Net-(C301-Pad2): track 0.00 -> 19.7 mm, vias 0 -> 1
- net Net-(C401-Pad2): track 0.00 -> 17.3 mm, vias 0 -> 1
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Other:
- board size 60 x 25 mm -> 60 x 16 mm
- board text added: "1"
- board text added: "2"
- board text added: "2.1-16v"
- board text added: "3"
- board text added: "4"
- board text added: "5.25.2015"
- board text added: "Brooke Hedrick"
- board text added: "Creative Commons: CC-BY"
- board text added: "DasBlinkInput : dbi_v1"
- board text added: "GND"
- board text added: "Out"
- board text added: "brooke.t.hedrick@gmail.com"
- board text added: "https://github.com/hedrickbt/ContextualElectronics.git"
