File: DasBlinkInput/pcb/Channel3Photodetect.sch (KiCad schematic (older format))
At the start: 6 parts, among them P401 TP_CHAN3, U201 MCP6404, U202 LM339

Commit message: DBI - fixed reg/on pin, changed resistor to 0 ohm near divider and rv, added 10k pull up resistors to 3V for each output channel.
Parts:
- added R402: 10K, Resistors_SMD:R_0805_HandSoldering, symbol R
Connections:
- net CHAN3_OUT: now also R402.2
- new net 3V: R402.1
Other:
- note added: "v2"
Changed lines of the file:
@@
 	6150 2650 6150 2850
 Connection ~ 6150 2850
+Text Notes 10600 7650 0    60   ~ 0
+v2
+$Comp
+L R R402
+U 1 1 55B59FDD
+P 8000 2550
+F 0 "R402" V 8080 2550 50  0000 C CNN
+F 1 "10K" V 8007 2551 50  0000 C CNN
+F 2 "Resistors_SMD:R_0805_HandSoldering" V 7930 2550 30  0001 C CNN
+F 3 "" H 8000 2550 30  0000 C CNN
+	1    8000 2550
+	1    0    0    -1
+$EndComp
+Text GLabel 7550 2150 0    60   Input ~ 0
+3V
+Wire Wire Line
+	7550 2150 8000 2150
+Wire Wire Line
+	8000 2150 8000 2300
+Wire Wire Line
+	8000 2800 8000 2950
+Connection ~ 8000 2950
 $EndSCHEMATC
