File: DasBlinkInput/pcb/DasBlinkInput.sch (KiCad schematic (older format))
At the start: 10 parts

Commit message: Progress on DBI schematic
Parts:
- removed C? (x3): C, symbol C
- removed D?: Photodiode, symbol Photodiode
- removed R? (x3): R, symbol R
- removed RV?: POT, symbol POT
- removed U?: MCP6404-E/SL, symbol MCP6404-E/SL
- removed U?: LM339, symbol LM339
- added C101, C102: 1uf, Capacitors_SMD:C_0805_HandSoldering, symbol C
- added P101: CONN_01X02, Pin_Headers:Pin_Header_Straight_1x02, symbol CONN_01X02
- added P102: TP_VGND, pcb:TESTPOINT_1, symbol CONN_01X01
- added P103: TP_GND, pcb:TESTPOINT_1, symbol CONN_01X01
- added P104: TP_3V, pcb:TESTPOINT_1, symbol CONN_01X01
- added P105: CONN_01X05, Pin_Headers:Pin_Header_Straight_1x05, symbol CONN_01X05
- added R101, R102: 10K, Resistors_SMD:R_0805_HandSoldering, symbol R
- added R103: 0, Resistors_SMD:R_0805_HandSoldering, symbol R
- added U101: LP2980-N, Housings_SOT-23_SOT-143_TSOT-6:SOT-23-5, symbol LP2980-N
Connections:
- net 3V: now also C102.1, P104.1 (P1), R101.1, U101.5 (OUT)
- net GND: now also C101.2, C102.2, P101.1 (P1), P103.1 (P1), P105.5 (P5), R102.2, R103.2, U101.2 (GND)
- new net: C101.1, P101.2 (P2), U101.1 (IN)
- new net: R103.1, U101.3 (ON/~OFF)
- new net Channel1Photodetect/CHAN1_OUT: P105.1 (P1)
- new net Channel2Photodetect/CHAN2_OUT: P105.2 (P2)
- new net Channel3Photodetect/CHAN3_OUT: P105.3 (P3)
- new net Channel4Photodetect/CHAN4_OUT: P105.4 (P4)
- new net VGND: P102.1 (P1), R101.2, R102.1
- no-connect marks 0 -> 1

Commit message: DBI : complete pcb
Parts:
- added P106: VREF, pcb:TESTPOINT_1, symbol CONN_01X01
Connections:
- net Channel1Photodetect/REF_OUT: now also P106.1 (P1)
Changed lines of the file:
@@
 	7400 1850 7400 2200
 $Comp
-L GND #PWR104
+L GND #PWR01
 U 1 1 555ABC4A
 P 7400 2200
-F 0 "#PWR104" H 7400 1950 60  0001 C CNN
+F 0 "#PWR01" H 7400 1950 60  0001 C CNN
 F 1 "GND" H 7400 2050 60  0000 C CNN
 F 2 "" H 7400 2200 60  0000 C CNN
@@
 	1250 1250 1250 1700
 $Comp
-L GND #PWR101
+L GND #PWR02
 U 1 1 555ABF20
 P 1250 1700
-F 0 "#PWR101" H 1250 1450 60  0001 C CNN
+F 0 "#PWR02" H 1250 1450 60  0001 C CNN
 F 1 "GND" H 1250 1550 60  0000 C CNN
 F 2 "" H 1250 1700 60  0000 C CNN
@@
 Connection ~ 2850 2100
 $Comp
-L GND #PWR103
+L GND #PWR03
 U 1 1 555AD295
 P 2850 2400
-F 0 "#PWR103" H 2850 2150 60  0001 C CNN
+F 0 "#PWR03" H 2850 2150 60  0001 C CNN
 F 1 "GND" H 2850 2250 60  0000 C CNN
 F 2 "" H 2850 2400 60  0000 C CNN
@@
 $EndComp
 $Comp
-L GND #PWR102
+L GND #PWR04
 U 1 1 555AD36F
 P 1450 4450
-F 0 "#PWR102" H 1450 4200 60  0001 C CNN
+F 0 "#PWR04" H 1450 4200 60  0001 C CNN
 F 1 "GND" H 1450 4300 60  0000 C CNN
 F 2 "" H 1450 4450 60  0000 C CNN
@@
 	3300 2400 3300 2100
 Connection ~ 3300 2100
+$Comp
+L CONN_01X01 P106
+U 1 1 556346E5
+P 3950 3650
+F 0 "P106" H 3950 3750 50  0000 C CNN
+F 1 "VREF" V 4050 3650 50  0000 C CNN
+F 2 "pcb:TESTPOINT_1" H 3950 3650 60  0001 C CNN
+F 3 "" H 3950 3650 60  0000 C CNN
+	1    3950 3650
+	0    -1   -1   0
+$EndComp
+Wire Wire Line
+	3950 3850 4350 3850
+Connection ~ 4350 3850
 $EndSCHEMATC

Commit message: DBI - fixed reg/on pin, changed resistor to 0 ohm near divider and rv, added 10k pull up resistors to 3V for each output channel.
Connections:
- net GND: no longer R103.2
- net at C101.1, P101.2 (P2), U101.1 (IN): now also R103.1
- net at U101.3 (ON/~OFF): now also R103.2; no longer R103.1
Other:
- note added: "v2"
- moved on the sheet: C101, P101, R103
Changed lines of the file:
@@
 L CONN_01X02 P101
 U 1 1 555ABEBF
-P 900 1200
-F 0 "P101" H 900 1350 50  0000 C CNN
-F 1 "CONN_01X02" V 1000 1200 50  0000 C CNN
-F 2 "Pin_Headers:Pin_Header_Straight_1x02" H 900 1200 60  0001 C CNN
-F 3 "" H 900 1200 60  0000 C CNN
-	1    900  1200
+P 650 1200
+F 0 "P101" H 550 1350 50  0000 C CNN
+F 1 "CONN_01X02" V 750 1200 50  0000 C CNN
+F 2 "Pin_Headers:Pin_Header_Straight_1x02" H 650 1200 60  0001 C CNN
+F 3 "" H 650 1200 60  0000 C CNN
+	1    650  1200
 	-1   0    0    1
 $EndComp
 Wire Wire Line
-	1100 1250 1250 1250
-Wire Wire Line
-	1250 1250 1250 1700
+	850  1250 1000 1250
+Wire Wire Line
+	1000 1250 1000 1700
 $Comp
 L GND #PWR02
 U 1 1 555ABF20
-P 1250 1700
-F 0 "#PWR02" H 1250 1450 60  0001 C CNN
-F 1 "GND" H 1250 1550 60  0000 C CNN
-F 2 "" H 1250 1700 60  0000 C CNN
-F 3 "" H 1250 1700 60  0000 C CNN
-	1    1250 1700
-	1    0    0    -1
-$EndComp
-Wire Wire Line
-	1100 1150 1900 1150
+P 1000 1700
+F 0 "#PWR02" H 1000 1450 60  0001 C CNN
+F 1 "GND" H 1000 1550 60  0000 C CNN
+F 2 "" H 1000 1700 60  0000 C CNN
+F 3 "" H 1000 1700 60  0000 C CNN
+	1    1000 1700
+	1    0    0    -1
+$EndComp
+Wire Wire Line
+	850  1150 1900 1150
 $Comp
 L LP2980-N U101
@@
 L C C101
 U 1 1 555AC341
-P 1450 1500
-F 0 "C101" H 1500 1600 50  0000 L CNN
-F 1 "1uf" H 1500 1400 50  0000 L CNN
-F 2 "Capacitors_SMD:C_0805_HandSoldering" H 1488 1350 30  0001 C CNN
-F 3 "" H 1450 1500 60  0000 C CNN
-F 4 "Value" H 1450 1500 60  0001 C CNN "MPN"
-	1    1450 1500
-	1    0    0    -1
-$EndComp
-Wire Wire Line
-	1450 2100 3450 2100
+P 1300 1500
+F 0 "C101" H 1350 1600 50  0000 L CNN
+F 1 "1uf" H 1350 1400 50  0000 L CNN
+F 2 "Capacitors_SMD:C_0805_HandSoldering" H 1338 1350 30  0001 C CNN
+F 3 "" H 1300 1500 60  0000 C CNN
+F 4 "Value" H 1300 1500 60  0001 C CNN "MPN"
+	1    1300 1500
+	1    0    0    -1
+$EndComp
+Wire Wire Line
+	1300 2100 3450 2100
 Wire Wire Line
 	2600 2100 2600 1950
@@
 	1    0    0    -1
 $EndComp
-Wire Wire Line
-	1450 1700 1450 2100
-Wire Wire Line
-	1450 1300 1450 1150
-Connection ~ 1450 1150
 $Comp
 L R R103
 U 1 1 555AC8F0
-P 1750 1750
-F 0 "R103" V 1830 1750 50  0000 C CNN
-F 1 "0" V 1757 1751 50  0000 C CNN
-F 2 "Resistors_SMD:R_0805_HandSoldering" V 1680 1750 30  0001 C CNN
-F 3 "" H 1750 1750 30  0000 C CNN
-F 4 "Value" H 1750 1750 60  0001 C CNN "MPN"
-	1    1750 1750
-	1    0    0    -1
-$EndComp
-Wire Wire Line
-	1900 1350 1750 1350
-Wire Wire Line
-	1750 1350 1750 1500
-Wire Wire Line
-	1750 2000 1750 2100
-Connection ~ 1750 2100
+P 1650 1500
+F 0 "R103" V 1730 1500 50  0000 C CNN
+F 1 "0" V 1657 1501 50  0000 C CNN
+F 2 "Resistors_SMD:R_0805_HandSoldering" V 1580 1500 30  0001 C CNN
+F 3 "" H 1650 1500 30  0000 C CNN
+F 4 "Value" H 1650 1500 60  0001 C CNN "MPN"
+	1    1650 1500
+	1    0    0    -1
+$EndComp
 NoConn ~ 1900 1550
 Wire Wire Line
@@
 	3950 3850 4350 3850
 Connection ~ 4350 3850
+Wire Wire Line
+	1300 1300 1300 1150
+Connection ~ 1300 1150
+Wire Wire Line
+	1300 1700 1300 2100
+Wire Wire Line
+	1650 1750 1650 1800
+Wire Wire Line
+	1650 1800 1800 1800
+Wire Wire Line
+	1800 1800 1800 1350
+Wire Wire Line
+	1800 1350 1900 1350
+Wire Wire Line
+	1650 1250 1650 1150
+Connection ~ 1650 1150
+Text Notes 10600 7650 0    60   ~ 0
+v2
 $EndSCHEMATC
