File: GoGoGo/pcb/MotorEncoder/MotorEncoder.kicad_pcb (KiCad board)
At the start: 2 copper layers, 19.2 x 17.9 mm, 11 parts, among them P101 CONN_01X02, P102 OPTO_OUT, P103 CONN_01X02, U101 RPI-579N1, U102 LM311DR

Commit message: GGG : Motor Encoder : changed R102 to 10K and started v2
Parts:
- R102: value 1K -> 10K
Other:
- board text added: "brooke.t.hedrick@gmail.com GGG MotorEncoder v2 License: CCBY github: hedrickbt/ContextualElectronics/ tree/master/GoGoGo"
- board text removed: "brooke.t.hedrick@gmail.com GGG MotorEncoder v1 License: CCBY github: hedrickbt/ContextualElectronics/ tree/master/GoGoGo"
