File: PowerSwap/pcb/PowerSwap.sch (KiCad schematic (older format))
At the start: 17 parts, among them P101 INPUT, P102 TP B4L, P103 TP FB, P104 TP AFTL, P105 TP VOUT1, P106 TP VOUT2, P107 OUTPUT, U101 TPS63030

Commit message: PS : starting inductor footprint
Parts:
- C101: value 4.7/10uf -> 4.7uf
- C103: value 10uf -> 22uf
- L101: value INDUCTOR -> 2.2uh; MPN (none) -> LQH3NPN2R2NG0
- R104: value R -> 1.2M; MPN (none) -> Value
- R105: value R -> 215K
Changed lines of the file:
@@
 P 4150 2200
 F 0 "L101" V 4100 2200 50  0000 C CNN
-F 1 "INDUCTOR" V 4250 2200 50  0000 C CNN
+F 1 "2.2uh" V 4250 2200 50  0000 C CNN
 F 2 "" H 4150 2200 60  0001 C CNN
 F 3 "" H 4150 2200 60  0000 C CNN
+F 4 "LQH3NPN2R2NG0" H 4150 2200 60  0001 C CNN "MPN"
 	1    4150 2200
 	0    -1   -1   0
@@
 P 1600 3200
 F 0 "C101" H 1650 3300 50  0000 L CNN
-F 1 "4.7/10uf" H 1650 3100 50  0000 L CNN
+F 1 "4.7uf" H 1650 3100 50  0000 L CNN
 F 2 "" H 1638 3050 30  0001 C CNN
 F 3 "" H 1600 3200 60  0000 C CNN
@@
 P 5550 3250
 F 0 "C103" H 5600 3350 50  0000 L CNN
-F 1 "10uf" H 5600 3150 50  0000 L CNN
+F 1 "22uf" H 5600 3150 50  0000 L CNN
 F 2 "" H 5588 3100 30  0001 C CNN
 F 3 "" H 5550 3250 60  0000 C CNN
@@
 P 5300 3200
 F 0 "R104" V 5380 3200 50  0000 C CNN
-F 1 "R" V 5307 3201 50  0000 C CNN
+F 1 "1.2M" V 5307 3201 50  0000 C CNN
 F 2 "" V 5230 3200 30  0001 C CNN
 F 3 "" H 5300 3200 30  0000 C CNN
+F 4 "Value" H 5300 3200 60  0001 C CNN "MPN"
 	1    5300 3200
 	1    0    0    -1
@@
 P 5300 3900
 F 0 "R105" V 5380 3900 50  0000 C CNN
-F 1 "R" V 5307 3901 50  0000 C CNN
+F 1 "215K" V 5307 3901 50  0000 C CNN
 F 2 "" V 5230 3900 30  0001 C CNN
 F 3 "" H 5300 3900 30  0000 C CNN

Commit message: PS : working on regulator footprint
Parts:
- L101: footprint (none) -> pcb:LQH3NPN2R2NG0
- U101: footprint (none) -> pcb:SON10_HandSoldered_TPS63030
Changed lines of the file:
@@
 F 0 "U101" H 4150 2450 60  0000 C CNN
 F 1 "TPS63030" H 4150 3750 60  0000 C CNN
-F 2 "" H 4150 3150 60  0001 C CNN
+F 2 "pcb:SON10_HandSoldered_TPS63030" H 4150 3150 60  0001 C CNN
 F 3 "" H 4150 3150 60  0000 C CNN
 	1    4150 3150
@@
 F 0 "L101" V 4100 2200 50  0000 C CNN
 F 1 "2.2uh" V 4250 2200 50  0000 C CNN
-F 2 "" H 4150 2200 60  0001 C CNN
+F 2 "pcb:LQH3NPN2R2NG0" H 4150 2200 60  0001 C CNN
 F 3 "" H 4150 2200 60  0000 C CNN
 F 4 "LQH3NPN2R2NG0" H 4150 2200 60  0001 C CNN "MPN"

Commit message: PS : associate and start pcb
Parts:
- added C104: uf, Capacitors_SMD:C_0805_HandSoldering, symbol C
- C101, C102: footprint (none) -> Capacitors_SMD:C_0805_HandSoldering
- C103: footprint (none) -> Capacitors_SMD:C_1210_HandSoldering
- P101, P107: footprint (none) -> Pin_Headers:Pin_Header_Straight_1x02
- P102, P103, P104, P105, P106: footprint (none) -> pcb:TESTPOINT_1
- R101, R102, R103, R104, R105: footprint (none) -> Resistors_SMD:R_0805_HandSoldering
Connections:
- net GNDPWR: now also C104.2
- net VOUT+: now also C104.1
Other:
- note added: "May be nopop"
Changed lines of the file:
@@
 F 0 "C101" H 1650 3300 50  0000 L CNN
 F 1 "4.7uf" H 1650 3100 50  0000 L CNN
-F 2 "" H 1638 3050 30  0001 C CNN
+F 2 "Capacitors_SMD:C_0805_HandSoldering" H 1638 3050 30  0001 C CNN
 F 3 "" H 1600 3200 60  0000 C CNN
 F 4 "Value" H 1600 3200 60  0001 C CNN "MPN"
@@
 F 0 "C103" H 5600 3350 50  0000 L CNN
 F 1 "22uf" H 5600 3150 50  0000 L CNN
-F 2 "" H 5588 3100 30  0001 C CNN
+F 2 "Capacitors_SMD:C_1210_HandSoldering" H 5588 3100 30  0001 C CNN
 F 3 "" H 5550 3250 60  0000 C CNN
 F 4 "Value" H 5550 3250 60  0001 C CNN "MPN"
@@
 F 0 "P107" H 6500 3350 50  0000 C CNN
 F 1 "OUTPUT" V 6600 3200 50  0000 C CNN
-F 2 "" H 6500 3200 60  0001 C CNN
+F 2 "Pin_Headers:Pin_Header_Straight_1x02" H 6500 3200 60  0001 C CNN
 F 3 "" H 6500 3200 60  0000 C CNN
 	1    6500 3200
 	1    0    0    -1
 $EndComp
-Text Label 5900 2850 0    60   ~ 0
+Text Label 6000 2850 0    60   ~ 0
 VOUT+
-Text Label 5900 3550 0    60   ~ 0
+Text Label 6000 3650 0    60   ~ 0
 VOUT-
 $Comp
@@
 F 0 "P101" H 1200 3350 50  0000 C CNN
 F 1 "INPUT" V 1300 3200 50  0000 C CNN
-F 2 "" H 1200 3200 60  0001 C CNN
+F 2 "Pin_Headers:Pin_Header_Straight_1x02" H 1200 3200 60  0001 C CNN
 F 3 "" H 1200 3200 60  0000 C CNN
 	1    1200 3200
@@
 F 0 "R104" V 5380 3200 50  0000 C CNN
 F 1 "1.2M" V 5307 3201 50  0000 C CNN
-F 2 "" V 5230 3200 30  0001 C CNN
+F 2 "Resistors_SMD:R_0805_HandSoldering" V 5230 3200 30  0001 C CNN
 F 3 "" H 5300 3200 30  0000 C CNN
 F 4 "Value" H 5300 3200 60  0001 C CNN "MPN"
@@
 F 0 "R105" V 5380 3900 50  0000 C CNN
 F 1 "215K" V 5307 3901 50  0000 C CNN
-F 2 "" V 5230 3900 30  0001 C CNN
+F 2 "Resistors_SMD:R_0805_HandSoldering" V 5230 3900 30  0001 C CNN
 F 3 "" H 5300 3900 30  0000 C CNN
 	1    5300 3900
@@
 F 0 "P103" H 4950 3250 50  0000 C CNN
 F 1 "TP FB" V 5050 3150 50  0000 C CNN
-F 2 "" H 4950 3150 60  0001 C CNN
+F 2 "pcb:TESTPOINT_1" H 4950 3150 60  0001 C CNN
 F 3 "" H 4950 3150 60  0000 C CNN
 	1    4950 3150
@@
 F 0 "P102" H 3300 2150 50  0000 C CNN
 F 1 "TP B4L" V 3400 2050 50  0000 C CNN
-F 2 "" H 3300 2050 60  0001 C CNN
+F 2 "pcb:TESTPOINT_1" H 3300 2050 60  0001 C CNN
 F 3 "" H 3300 2050 60  0000 C CNN
 	1    3300 2050
@@
 F 0 "P104" H 5050 2200 50  0000 C CNN
 F 1 "TP AFTL" V 5150 2100 50  0000 C CNN
-F 2 "" H 5050 2100 60  0001 C CNN
+F 2 "pcb:TESTPOINT_1" H 5050 2100 60  0001 C CNN
 F 3 "" H 5050 2100 60  0000 C CNN
 	1    5050 2100
@@
 F 0 "P105" H 5250 2500 50  0000 C CNN
 F 1 "TP VOUT1" V 5350 2400 50  0000 C CNN
-F 2 "" H 5250 2400 60  0001 C CNN
+F 2 "pcb:TESTPOINT_1" H 5250 2400 60  0001 C CNN
 F 3 "" H 5250 2400 60  0000 C CNN
 	1    5250 2400
@@
 F 0 "P106" H 5700 2500 50  0000 C CNN
 F 1 "TP VOUT2" V 5800 2400 50  0000 C CNN
-F 2 "" H 5700 2400 60  0001 C CNN
+F 2 "pcb:TESTPOINT_1" H 5700 2400 60  0001 C CNN
 F 3 "" H 5700 2400 60  0000 C CNN
 	1    5700 2400
@@
 F 0 "R101" V 2480 3050 50  0000 C CNN
 F 1 "0" V 2407 3051 50  0000 C CNN
-F 2 "" V 2330 3050 30  0001 C CNN
+F 2 "Resistors_SMD:R_0805_HandSoldering" V 2330 3050 30  0001 C CNN
 F 3 "" H 2400 3050 30  0000 C CNN
 F 4 "Value" H 2400 3050 60  0001 C CNN "MPN"
@@
 F 0 "R102" V 3230 3250 50  0000 C CNN
 F 1 "0" V 3157 3251 50  0000 C CNN
-F 2 "" V 3080 3250 30  0001 C CNN
+F 2 "Resistors_SMD:R_0805_HandSoldering" V 3080 3250 30  0001 C CNN
 F 3 "" H 3150 3250 30  0000 C CNN
 	1    3150 3250
@@
 F 0 "R103" V 3230 3450 50  0000 C CNN
 F 1 "0" V 3157 3451 50  0000 C CNN
-F 2 "" V 3080 3450 30  0001 C CNN
+F 2 "Resistors_SMD:R_0805_HandSoldering" V 3080 3450 30  0001 C CNN
 F 3 "" H 3150 3450 30  0000 C CNN
 	1    3150 3450
@@
 F 0 "C102" H 2450 3950 50  0000 L CNN
 F 1 "0.1uf" H 2450 3750 50  0000 L CNN
-F 2 "" H 2438 3700 30  0001 C CNN
+F 2 "Capacitors_SMD:C_0805_HandSoldering" H 2438 3700 30  0001 C CNN
 F 3 "" H 2400 3850 60  0000 C CNN
 F 4 "Value" H 2400 3850 60  0001 C CNN "MPN"
@@
 	3400 3650 3400 3950
 Connection ~ 3400 3950
+$Comp
+L C C104
+U 1 1 55CFB4F6
+P 5900 3250
+F 0 "C104" H 5950 3350 50  0000 L CNN
+F 1 "uf" H 5950 3150 50  0000 L CNN
+F 2 "Capacitors_SMD:C_0805_HandSoldering" H 5938 3100 30  0001 C CNN
+F 3 "" H 5900 3250 60  0000 C CNN
+F 4 "Value" H 5900 3250 60  0001 C CNN "MPN"
+	1    5900 3250
+	1    0    0    -1
+$EndComp
+Wire Wire Line
+	5900 3050 5900 2850
+Connection ~ 5900 2850
+Wire Wire Line
+	5900 3450 5900 3550
+Connection ~ 5900 3550
+Text Notes 6100 3550 1    60   ~ 0
+May be nopop
 $EndSCHEMATC
