File: PowerSwap/pcb/PowerSwap.kicad_pcb (KiCad board)
At the start: 2 copper layers, 0 parts

Commit message: PS : associate and start pcb
Parts:
- added C101: 4.7uf, Capacitors_SMD:C_0805_HandSoldering, F.Cu at (151.8, 98.8)
- added C102: 0.1uf, Capacitors_SMD:C_0805_HandSoldering, F.Cu at (151.8, 105.2)
- added C103: 22uf, Capacitors_SMD:C_1210_HandSoldering, F.Cu at (158.4, 95.3)
- added C104: uf, Capacitors_SMD:C_0805_HandSoldering, F.Cu at (157.0, 102.3)
- added L101: 2.2uh, pcb:LQH3NPN2R2NG0, F.Cu at (151.2, 91.0)
- added P101: INPUT, Pin_Headers:Pin_Header_Straight_1x02, F.Cu at (145.4, 92.4)
- added P102: TP B4L, pcb:TESTPOINT_1, F.Cu at (170.2, 101.7)
- added P103: TP FB, pcb:TESTPOINT_1, F.Cu at (167.3, 106.9)
- added P104: TP AFTL, pcb:TESTPOINT_1, F.Cu at (165.1, 94.1)
- added P105: TP VOUT1, pcb:TESTPOINT_1, F.Cu at (166.5, 88.9)
- added P106: TP VOUT2, pcb:TESTPOINT_1, F.Cu at (158.7, 88.9)
- added P107: OUTPUT, Pin_Headers:Pin_Header_Straight_1x02, F.Cu at (146.1, 103.3)
- added R101: 0, Resistors_SMD:R_0805_HandSoldering, F.Cu at (173.2, 89.4)
- added R102: 0, Resistors_SMD:R_0805_HandSoldering, F.Cu at (164.7, 99.9)
- added R103: 0, Resistors_SMD:R_0805_HandSoldering, F.Cu at (171.1, 95.8)
- added R104: 1.2M, Resistors_SMD:R_0805_HandSoldering, F.Cu at (178.6, 89.4)
- added R105: 215K, Resistors_SMD:R_0805_HandSoldering, F.Cu at (162.2, 106.3)
- added U101: TPS63030, pcb:SON10_HandSoldered_TPS63030, F.Cu at (176.1, 95.6)

Commit message: PS : first layout complete and gerbers generated
Parts:
- moved R104 33.1 mm to (163.9, 119.1)
- moved P107 31.1 mm to (174.7, 115.5)
- moved P106 31.0 mm to (171.4, 117.1)
- moved R101 30.5 mm to (152.0, 111.4)
- moved R103 27.6 mm to (152.0, 115.7), turned to 180 degrees
- moved U101 27.0 mm to (159.6, 117.0), turned to 270 degrees
- moved P105 25.6 mm to (162.1, 114.1)
- moved L101 22.0 mm to (159.7, 111.3), turned to 90 degrees
- moved C103 19.7 mm to (166.7, 113.2)
- moved C104 18.6 mm to (171.6, 113.9), turned to 90 degrees
- moved R102 18.6 mm to (152.0, 113.5), turned to 180 degrees
- moved P101 17.3 mm to (152.6, 108.2), turned to 270 degrees
- moved C102 15.1 mm to (155.5, 119.9), turned to 180 degrees
- moved P104 15.0 mm to (160.9, 108.5)
- moved R105 14.7 mm to (169.6, 119.0)
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Routing:
- net /VOUT+: track 0.00 -> 34.2 mm
- net GNDPWR: track 0.00 -> 20.5 mm, vias 0 -> 6
- net Net-(C102-Pad1): track 0.00 -> 16.6 mm
- net Net-(P103-Pad1): track 0.00 -> 15.3 mm
- net Net-(R103-Pad1): track 0.00 -> 8.83 mm
- net Net-(R102-Pad1): track 0.00 -> 8.67 mm
- net Net-(L101-Pad2): track 0.00 -> 7.33 mm
- net Net-(L101-Pad1): track 0.00 -> 7.23 mm
- added copper zone on F.Cu, net /VIN+
- added copper zone on B.Cu, net GNDPWR
Other:
- board outline added: 29.2 x 17.2 mm
- net class Default: clearance 0.254 -> 0.1524; trace_width 0.254 -> 0.1524; via_dia 0.889 -> 0.6858; via_drill 0.635 -> 0.3302
- net class PWR added: clearance 0.1524, trace_width 0.6096, via_dia 0.6858, via_drill 0.3302
- rule trace_clearance: 0.254 -> 0.1524
- rule trace_min: 0.254 -> 0.1524
- rule via_min_drill: 0.508 -> 0.3302
- rule via_min_size: 0.889 -> 0.6858
- board text added: "+"
- board text added: "-"
- board text added: "3.3V Output"
- board text added: "3.6-5.5v Input"
- board text added: "?"
- board text added: "License: CCBY"
- board text added: "PowerSwap v1"
- board text added: "brooke.t.hedrick@gmail.com"
- board text added: "github hedrickbt ContextualElectronics/PowerSwap"

Commit message: PS : small pcb change
Routing:
- net GNDPWR: track 20.5 -> 19.9 mm, vias 6 -> 5
